File: hw/sch_pcb/SOLARMINIBAT01A.kicad_sch (KiCad schematic)
At the start: 6 parts, among them J7 JUMP_4X2, J8 CONN1_1, J9 CONN1_1

Commit message: Pridano schema menice ze solarniho clanku
Other:
- added sheet solar_converter (solar_converter.kicad_sch)
