File: hw/sch_pcb/SOLARMINIBAT01A.kicad_pcb (KiCad board)
At the start: 2 copper layers, 80.8 x 60.5 mm, 100 parts, among them J1 JUMP_4X2, J10 JUMP_2x1, J11 JUMP_2x1, J12 JUMP_2x1, J13 JUMP_4X2, J14 JUMP_2x1, J15 CONN_2, J2 JUMP_2x1, J3 JUMP_2x1, J4 JUMP2_2x1, J5 JUMP_2x1, J6 JUMP_2x1, J7 JUMP_4X2, J8 CONN1_1, J9 CONN1_1, P1 _, P2 _, P3 _, P4 _, Q1 IRLML6244, SW1 SW_PUSH, U1 BQ29209, U2 BQ24103, U3 BQ34Z100, U4 SN74HC164D, U5 TPS76601, U6 APX810-31SAG-7

Commit message: Edit schema
Parts:
- removed BT1: 2x18650_LION-RESCUE-LION2CELL01C, Mlab_Batery:2LION
- removed D11, D12, D13, D14: ORAGE, Mlab_D:LED_1206
- removed F3: 2A, Mlab_F:Drzak_2410
- removed J10, J11, J12, J14: JUMP_2x1, Mlab_Pin_Headers:Straight_1x02
- removed J13, J7: JUMP_4X2, Mlab_Pin_Headers:Straight_2x04
- removed J15: CONN_2, Mlab_Pin_Headers:SMD_1_2x2
- removed J8, J9: CONN1_1, Mlab_Con:WAGO256
- removed P2, P3, P4: _, Mlab_Mechanical:MountingHole_3mm
- removed Q1: IRLML6244, Mlab_T:SOT-23
- removed R27, R28, R29, R30, R31, R32, R33, R34: 2K2, Mlab_R:SMD-0805
- removed R35, R36: 47k, Mlab_R:SMD-0805
- removed U4: SN74HC164D, Mlab_IO:SO-14
- removed U5: TPS76601, Mlab_IO:SO-8
- removed U6: APX810-31SAG-7, Mlab_IO:SOT-23
- added C21: 47uF/6V3, Capacitor_SMD:C_0805_2012Metric, F.Cu at (181.6, 61.9)
- added C22: 47uF/6V3, Capacitor_SMD:C_0805_2012Metric, F.Cu at (177.1, 61.9)
- added D6: ORAGE, Mlab_D:LED_1206, F.Cu at (108.3, 81.3)
- added JP1: SolderJumper_2_Open, Jumper:SolderJumper-2_P1.3mm_Open_RoundedPad1.0x1.5mm, F.Cu at (166.5, 73.3)
- added L2: DE1207-1, Mlab_L:DE1205-10, F.Cu at (161.6, 64.5)
- added M1: HOLE, Mlab_Mechanical:MountingHole_3mm, F.Cu at (156.3, 90.1)
- added M2: HOLE, Mlab_Mechanical:MountingHole_3mm, F.Cu at (156.3, 97.5)
- added M3: HOLE, Mlab_Mechanical:MountingHole_3mm, F.Cu at (163.6, 90.1)
- added M4: HOLE, Mlab_Mechanical:MountingHole_3mm, F.Cu at (163.6, 97.5)
- added X1: TPS63060, Package_SON:Texas_S-PWSON-N10_ThermalVias, F.Cu at (157.2, 74.1)
- C1, C12, C18, C4, C6, C7, C9: footprint Mlab_R:SMD-0805 -> Capacitor_SMD:C_0805_2012Metric; moved to F.Cu
- C10: value 100uF -> 1uF; footprint Mlab_C:TantalC_SizeD_Reflow -> Capacitor_SMD:C_0805_2012Metric; moved to F.Cu
- C11: value 10uF -> 1nF; footprint Mlab_R:SMD-0805 -> Capacitor_SMD:C_0805_2012Metric; moved to F.Cu
- C13: value 100nF -> 10uF; footprint Mlab_R:SMD-0805 -> Capacitor_SMD:C_0805_2012Metric; moved to F.Cu
- C14: value 1uF -> 47uF/6V3; footprint Mlab_R:SMD-0805 -> Capacitor_SMD:C_0805_2012Metric; moved to F.Cu
- C15, C16, C8: value 100nF -> 47uF/6V3; footprint Mlab_R:SMD-0805 -> Capacitor_SMD:C_0805_2012Metric; moved to F.Cu
- C17: value 3n3 -> 10uF; footprint Mlab_R:SMD-0805 -> Capacitor_SMD:C_0805_2012Metric; moved to F.Cu
- C19: value 100nF -> 10pF; footprint Mlab_R:SMD-0805 -> Capacitor_SMD:C_0805_2012Metric; moved to F.Cu
- C2: value 47uF -> 1uF; footprint Mlab_C:TantalC_SizeC_Reflow -> Capacitor_SMD:C_0805_2012Metric; moved to F.Cu
- C20: value 10uF -> 10uF/6V3; footprint Mlab_C:TantalC_SizeC_Reflow -> Capacitor_SMD:C_0805_2012Metric; moved to F.Cu
- C3: value 10uF -> 100nF; footprint Mlab_R:SMD-0805 -> Capacitor_SMD:C_0805_2012Metric; moved to F.Cu
- C5: value 330nF -> 3n3; footprint Mlab_R:SMD-0805 -> Capacitor_SMD:C_0805_2012Metric; moved to F.Cu
- D1, D2: value M4 -> ORAGE; footprint Mlab_D:SMA_Standard -> Mlab_D:LED_1206; moved to F.Cu
- D10: value ORAGE -> SMBJ5.0A; footprint Mlab_D:LED_1206 -> Diode_SMD:D_SMA; moved to F.Cu
- D3, D4: value Green -> ORAGE; moved to F.Cu
- D5: value Red -> ORAGE; moved to F.Cu
- D7, D8: moved to F.Cu
- D9: value ORAGE -> 15MQ040N; footprint Mlab_D:LED_1206 -> Diode_SMD:D_SMA; moved to F.Cu
- F1: value 5A -> 1,1A; footprint Mlab_F:Drzak_2410 -> Fuse:Fuse_1812_4532Metric_Pad1.30x3.40mm_HandSolder; moved to F.Cu
- J1: value JUMP_4X2 -> HEADER_2x03_PARALLEL; footprint Mlab_Pin_Headers:Straight_2x04 -> Mlab_Pin_Headers:Straight_2x03
- J2: value JUMP_2x1 -> WAGO 256 RED; footprint Mlab_Pin_Headers:Straight_1x02 -> Mlab_CON:WAGO256
- J3: value JUMP_2x1 -> WAGO 256 BLUE; footprint Mlab_Pin_Headers:Straight_1x02 -> Mlab_CON:WAGO256
- J4: value JUMP2_2x1 -> HEADER_2x01_PARALLEL; footprint Mlab_Pin_Headers:Straight_1x02 -> Mlab_Pin_Headers:Straight_2x01
- J5, J6: value JUMP_2x1 -> HEADER_2x03_PARALLEL; footprint Mlab_Pin_Headers:Straight_1x02 -> Mlab_Pin_Headers:Straight_2x03
- L1: value DE1205-10 -> 10uH - DE1205-10; moved to F.Cu
- P1: value _ -> HEADER_2x05_PARALLEL; footprint Mlab_Mechanical:MountingHole_3mm -> Mlab_Pin_Headers:Straight_2x05
- R1: value 160R -> 47k; footprint Mlab_R:SMD-0805 -> Resistor_SMD:R_0805_2012Metric; moved to F.Cu
- R10: value 1K -> 270R; footprint Mlab_R:SMD-0805 -> Resistor_SMD:R_0805_2012Metric; moved to F.Cu
- R11, R12: value 7K5 -> 270R; footprint Mlab_R:SMD-0805 -> Resistor_SMD:R_0805_2012Metric; moved to F.Cu
- R13: value 9K31 -> 270R; footprint Mlab_R:SMD-0805 -> Resistor_SMD:R_0805_2012Metric; moved to F.Cu
- R14: value 442K -> 270R; footprint Mlab_R:SMD-0805 -> Resistor_SMD:R_0805_2012Metric; moved to F.Cu
- R15: value NCP21XV103J03RA -> 270R; footprint Mlab_R:SMD-0805 -> Resistor_SMD:R_0805_2012Metric
- R16: value 0R1 -> 270R; footprint Resistors_SMD:R_2512 -> Resistor_SMD:R_0805_2012Metric; moved to F.Cu
- R17: value 10K NTC -> 1k; footprint Mlab_R:SMD-0805 -> Resistor_SMD:R_0805_2012Metric
- R18, R19: value 100R -> 1k; footprint Mlab_R:SMD-0805 -> Resistor_SMD:R_0805_2012Metric; moved to F.Cu
- R2: value 260R -> 47k; footprint Mlab_R:SMD-0805 -> Resistor_SMD:R_0805_2012Metric; moved to F.Cu
- R20: value 1K -> 1k; footprint Mlab_R:SMD-0805 -> Resistor_SMD:R_0805_2012Metric; moved to F.Cu
- R21: value 270k -> 0R47; footprint Mlab_R:SMD-0805 -> Resistor_SMD:R_1206_3216Metric; moved to F.Cu
- R22: value 0R01 75PPM -> 560k; footprint Mlab_R:SMD-2512 -> Resistor_SMD:R_0805_2012Metric; moved to F.Cu
- R23: value 16k5 25ppm -> 270k; footprint Mlab_R:SMD-0805 -> Resistor_SMD:R_0805_2012Metric; moved to F.Cu
- R24: value 140k .1% 25ppm -> 10k; footprint Mlab_R:SMD-0805 -> Resistor_SMD:R_0805_2012Metric; moved to F.Cu
- R25: value 270k -> 560k; footprint Mlab_R:SMD-0805 -> Resistor_SMD:R_0805_2012Metric; moved to F.Cu
- R26: value 165k -> 100k; footprint Mlab_R:SMD-0805 -> Resistor_SMD:R_0805_2012Metric; moved to F.Cu
- R3: value 100R -> 47k; footprint Mlab_R:SMD-0805 -> Resistor_SMD:R_0805_2012Metric; moved to F.Cu
- R4: value 10k -> 10K NTC; footprint Mlab_R:SMD-0805 -> Resistor_SMD:R_0805_2012Metric; moved to F.Cu
- R5: value 10K -> 1K; footprint Mlab_R:SMD-0805 -> Resistor_SMD:R_0805_2012Metric; moved to F.Cu
- R6, R7: value 2K2 -> 100R; footprint Mlab_R:SMD-0805 -> Resistor_SMD:R_0805_2012Metric; moved to F.Cu
- R8: value 2K2 -> 0R01 75PPM; footprint Mlab_R:SMD-0805 -> Resistor_SMD:R_2512_6332Metric_Pad1.40x3.35mm_HandSolder; moved to F.Cu
- R9: value 100R -> 270R; footprint Mlab_R:SMD-0805 -> Resistor_SMD:R_0805_2012Metric; moved to F.Cu
- U1: value BQ29209 -> BQ34Z100; footprint Mlab_IO:VSON-8 -> Mlab_IO:TSSOP-14_4.4x5mm_Pitch0.65mm; moved to F.Cu
- U2: value BQ24103 -> SN74HC164D; footprint Mlab_IO:VQFN-20 -> Package_SO:SO-14_3.9x8.65mm_P1.27mm; moved to F.Cu
- U3: value BQ34Z100 -> SPV1040; footprint Mlab_IO:TSSOP-14_4.4x5mm_Pitch0.65mm -> Package_SO:TSSOP-8_4.4x3mm_P0.65mm; moved to F.Cu
- moved J1 215.2 mm to (195.9, 61.8), turned to 0 degrees
- moved F1 213.4 mm to (202.6, 59.9)
- moved J6 181.4 mm to (171.8, 70.6)
- moved J4 177.7 mm to (125.1, 102.4), turned to 0 degrees
- moved C9 176.8 mm to (115.5, 107.8), turned to 0 degrees
- moved C8 175.7 mm to (130.5, 102.1), turned to 0 degrees
- moved J5 171.7 mm to (171.8, 61.8)
- moved R2 166.5 mm to (143.4, 65.8), turned to 0 degrees
- moved R6 166.4 mm to (142.3, 62.9), turned to 0 degrees
- moved C20 165.8 mm to (177.1, 64.9), turned to 0 degrees
- moved R12 164.9 mm to (148.5, 58.9), turned to 0 degrees
- moved R26 164.7 mm to (186.0, 61.9), turned to 0 degrees
- moved J2 164.4 mm to (113.2, 95.7)
- moved L1 164.1 mm to (130.9, 93.5), turned to 0 degrees
- moved D1 163.9 mm to (118.6, 74.9)
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Connections:
- C1 pad 1: Net-(C1-Pad1) -> +3V3
- C10 pad 2: GND -> Net-(C10-Pad2)
- C11 pad 1: Net-(C10-Pad1) -> Net-(C11-Pad1)
- C12 pad 1: +3V3 -> Net-(C12-Pad1)
- C13 pad 1: Net-(C13-Pad1) -> Net-(C12-Pad1)
- C13 pad 2: Net-(C13-Pad2) -> GND
- C14 pad 1: Net-(C14-Pad1) -> Net-(C12-Pad1)
- C15 pad 1: Net-(C13-Pad2) -> /battery_pack/Battery+
- C16 pad 1: Net-(C13-Pad1) -> /battery_pack/Battery+
- C17 pad 1: Net-(C17-Pad1) -> /battery_pack/Battery+
- C18 pad 1: +3V3 -> Net-(C18-Pad1)
- C19 pad 1: /BAT+ -> Net-(C19-Pad1)
- C3 pad 1: Net-(C2-Pad1) -> Net-(C3-Pad1)
- C3 pad 2: GND -> Net-(C3-Pad2)
- C4 pad 1: Net-(C4-Pad1) -> Net-(C3-Pad2)
- C4 pad 2: Net-(C1-Pad1) -> GND
- C5 pad 1: Net-(C5-Pad1) -> /battery_pack/Battery+
- C6 pad 1: /CMODE -> Net-(C3-Pad1)
- C7 pad 1: Net-(C2-Pad1) -> +3V3
- C8 pad 1: Net-(C8-Pad1) -> /power_input/PV+
- D1 pad 1: GND -> +3V3
- D1 pad 2: Net-(C2-Pad1) -> Net-(D1-Pad2)
- D10 pad 1: +3V3 -> Net-(C12-Pad1)
- D10 pad 2: Net-(D10-Pad2) -> GND
- D2 pad 1: GND -> +3V3
- D2 pad 2: /BATTERY+ -> Net-(D2-Pad2)
- D3 pad 1: Net-(D3-Pad1) -> +3V3
- D3 pad 2: /PG -> Net-(D3-Pad2)
- D4 pad 1: Net-(D4-Pad1) -> +3V3
- D4 pad 2: /STAT2 -> Net-(D4-Pad2)
- D5 pad 1: Net-(D5-Pad1) -> +3V3
- D5 pad 2: /STAT1 -> Net-(D5-Pad2)
- D9 pad 1: +3V3 -> Net-(C12-Pad1)
- F1 pad 1: /BAT+ -> /battery_pack/Battery+
- F1 pad 2: /BATTERY+ -> Net-(F1-Pad2)
- J1 pad 3: Net-(C2-Pad1) -> Net-(F1-Pad2)
- J1 pad 4: Net-(C2-Pad1) -> Net-(F1-Pad2)
- J1 pad 5: Net-(C2-Pad1) -> GND
- J1 pad 6: Net-(C2-Pad1) -> GND
- J2 pad 1: /STAT1 -> /power_input/PV+
- J3 pad 1: /PG -> GND
- J4 pad 1: /CMODE -> /fuel_gauge/CHARGE_CTRL
- J4 pad 2: GND -> /fuel_gauge/CHARGE_CTRL
- J5 pad 1: /CE -> GND
- J5 pad 2: /CE -> GND
- J6 pad 1: /STAT2 -> GND
- J6 pad 2: /STAT2 -> GND
- L1 pad 1: Net-(L1-Pad1) -> /power_input/PV+
- L1 pad 2: Net-(C10-Pad1) -> Net-(D9-Pad2)
- P1 pad 1: (no net) -> GND
- R1 pad 1: Net-(C4-Pad1) -> /fuel_gauge/I2C_SDA
- R1 pad 2: /BAT+ -> +3V3
- R10 pad 1: Net-(Q1-PadG) -> Net-(D2-Pad2)
- R11 pad 1: Net-(R11-Pad1) -> Net-(D3-Pad2)
- R11 pad 2: GND -> Net-(R11-Pad2)
- R12 pad 1: Net-(R12-Pad1) -> Net-(D4-Pad2)
- R12 pad 2: GND -> Net-(R12-Pad2)
- R13 pad 1: Net-(R13-Pad1) -> Net-(D5-Pad2)
- R13 pad 2: Net-(C9-Pad1) -> Net-(R13-Pad2)
- R14 pad 1: GND -> Net-(D6-Pad2)
- R14 pad 2: Net-(R13-Pad1) -> Net-(R14-Pad2)
- R15 pad 1: GND -> Net-(D7-Pad2)
- R15 pad 2: Net-(R13-Pad1) -> Net-(R15-Pad2)
- R16 pad 1: Net-(F3-Pad1) -> Net-(D8-Pad2)
- R16 pad 2: Net-(C10-Pad1) -> Net-(R16-Pad2)
- R17 pad 1: Net-(C14-Pad1) -> /power_input/PV+
- R17 pad 2: Net-(R17-Pad2) -> Net-(C9-Pad1)
- R18 pad 1: /BATTERY- -> /fuel_gauge/CHARGE_CTRL
- R18 pad 2: Net-(C13-Pad1) -> Net-(R18-Pad2)
- R19 pad 1: GND -> Net-(C10-Pad1)
- R19 pad 2: Net-(C13-Pad2) -> Net-(C12-Pad1)
- R2 pad 1: Net-(C1-Pad1) -> /fuel_gauge/CHARGE_CTRL
- R2 pad 2: /BAT-MIDPOINT -> +3V3
- R20 pad 1: Net-(R20-Pad1) -> Net-(C10-Pad2)
- R20 pad 2: Net-(C14-Pad1) -> /battery_pack/Battery+
- R21 pad 1: /CB_EN -> /battery_pack/Battery+
- R21 pad 2: Net-(C8-Pad1) -> Net-(C12-Pad1)
- R22 pad 1: /BATTERY- -> Net-(C11-Pad1)
- R22 pad 2: GND -> /battery_pack/Battery+
- R23 pad 2: Net-(C17-Pad1) -> Net-(C11-Pad1)
- R24 pad 1: /BAT+ -> /battery_pack/Battery+
- R24 pad 2: Net-(C17-Pad1) -> Net-(JP1-Pad2)
- R25 pad 1: Net-(R25-Pad1) -> +3V3
- R25 pad 2: +3V3 -> Net-(C19-Pad1)
- R26 pad 1: GND -> Net-(C19-Pad1)
- R26 pad 2: Net-(R25-Pad1) -> GND
- R3 pad 1: Net-(R3-Pad1) -> /fuel_gauge/I2C_SCL
- R3 pad 2: /BAT-MIDPOINT -> +3V3
- R4 pad 1: /CE -> Net-(C2-Pad1)
- R4 pad 2: GND -> Net-(R4-Pad2)
- R5 pad 1: Net-(C2-Pad1) -> Net-(R5-Pad1)
- R5 pad 2: Net-(R5-Pad2) -> Net-(C2-Pad1)
- R6 pad 1: Net-(C2-Pad1) -> /battery_pack/Battery-
- R6 pad 2: Net-(D3-Pad1) -> Net-(C3-Pad1)
- R7 pad 1: Net-(C2-Pad1) -> GND
- R7 pad 2: Net-(D4-Pad1) -> Net-(C3-Pad2)
- R8 pad 1: Net-(C2-Pad1) -> /battery_pack/Battery-
- R8 pad 2: Net-(D5-Pad1) -> GND
- R9 pad 1: Net-(C8-Pad1) -> Net-(D1-Pad2)
- R9 pad 2: /BAT+ -> Net-(R9-Pad2)
- SW1 pad 1: Net-(R20-Pad1) -> Net-(R5-Pad1)
- U1 pad 1: Net-(C4-Pad1) -> /fuel_gauge/P2
- U1 pad 2: Net-(C1-Pad1) -> Net-(SW1-Pad2)
- U1 pad 3: Net-(R3-Pad1) -> /fuel_gauge/P1
- U1 pad 4: Net-(C5-Pad1) -> /battery_pack/Battery+
- U1 pad 5: GND -> +3V3
- U1 pad 6: /CB_EN -> +3V3
- U1 pad 7: Net-(C8-Pad1) -> Net-(C2-Pad1)
- U1 pad 8: Net-(R10-Pad2) -> GND
- U1 pad 9: GND -> Net-(C3-Pad1)
- U2 pad 1: Net-(L1-Pad1) -> /fuel_gauge/P1
- U2 pad 10: GND -> Net-(R13-Pad2)
- U2 pad 11: Net-(C9-Pad1) -> Net-(R14-Pad2)
- U2 pad 12: Net-(R13-Pad1) -> Net-(R15-Pad2)
- U2 pad 13: Net-(R5-Pad2) -> Net-(R16-Pad2)
- U2 pad 14: Net-(F3-Pad1) -> +3V3
- U2 pad 2: /STAT1 -> /fuel_gauge/P1
- U2 pad 3: Net-(C2-Pad1) -> Net-(R9-Pad2)
- U2 pad 4: Net-(C2-Pad1) -> Net-(R10-Pad2)
- U2 pad 5: /PG -> Net-(R11-Pad2)
- U2 pad 6: Net-(C2-Pad1) -> Net-(R12-Pad2)
- U2 pad 7: /CMODE -> GND
- U2 pad 8: Net-(R12-Pad1) -> /fuel_gauge/P2
- U2 pad 9: Net-(R11-Pad1) -> +3V3
- U3 pad 1: /P2 -> Net-(C9-Pad1)
- U3 pad 2: Net-(SW1-Pad2) -> GND
- U3 pad 3: /P1 -> Net-(D9-Pad2)
- U3 pad 4: Net-(C17-Pad1) -> Net-(C12-Pad1)
- U3 pad 5: +3V3 -> Net-(C11-Pad1)
- U3 pad 6: +3V3 -> Net-(C10-Pad2)
- U3 pad 7: Net-(C14-Pad1) -> Net-(C10-Pad1)
- U3 pad 8: GND -> Net-(R18-Pad2)
Routing:
- net GND: track 726.1 -> 0.00 mm, vias 232 -> 0
- net /BAT+: track 124.9 -> 0.00 mm, vias 3 -> 0
- net +3V3: track 96.3 -> 0.00 mm, vias 4 -> 0
- net Net-(C10-Pad1): track 70.9 -> 0.00 mm, vias 2 -> 0
- net /STAT1: track 56.2 -> 0.00 mm, vias 2 -> 0
- net /PG: track 39.9 -> 0.00 mm, vias 2 -> 0
- net Net-(C2-Pad1): track 38.8 -> 0.00 mm
- net /SDA: track 35.8 -> 0.00 mm
- net /SCL: track 34.9 -> 0.00 mm
- net /HDQ: track 34.6 -> 0.00 mm
- net /STAT2: track 33.9 -> 0.00 mm, vias 2 -> 0
- net Net-(SW1-Pad2): track 31.4 -> 0.00 mm
- net /CMODE: track 31.3 -> 0.00 mm, vias 1 -> 0
- net /CE: track 31.0 -> 0.00 mm, vias 1 -> 0
- net Net-(R13-Pad1): track 28.6 -> 0.00 mm, vias 1 -> 0
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- removed copper zone on B.Cu, net +3V3
- removed copper zone on B.Cu, net /BAT+
- removed copper zone on B.Cu, net /BAT-MIDPOINT
- removed copper zone on F.Cu, net /BAT-MIDPOINT
- removed copper zone on B.Cu, net /BATTERY+
- removed copper zone on B.Cu, net /BATTERY-
- removed copper zone on B.Cu, net GND
- removed copper zone on F.Cu, net GND
- removed copper zone on B.Cu, net Net-(C10-Pad1)
- removed copper zone on B.Cu, net Net-(C2-Pad1)
- removed copper zone on B.Cu, net Net-(F3-Pad1)
- removed copper zone on B.Cu, net Net-(L1-Pad1)
Other:
- board outline removed
- board text removed: "+"
- board text removed: "0% ----100%"
- board text removed: "1"
- board text removed: "2"
- board text removed: "2016"
- board text removed: "3"
- board text removed: "4"
- board text removed: "5"
- board text removed: "6"
- board text removed: "CHARGE"
- board text removed: "DONE"
- board text removed: "GND"
- board text removed: "HDQ"
- board text removed: "JACHO"
- board text removed: "LION2CELL01D"
- board text removed: "MLAB.CZ"
- board text removed: "ON"
- board text removed: "POWER IN"
- board text removed: "POWER OUT"
- board text removed: "SCL"
- board text removed: "SDA"
- board text removed: "SW POWER"

Commit message: Edit PCB
Parts:
- added BT1: 4xLTO18650, Mlab_Batery:4XLTO1865V01A, F.Cu at (92.4, 116.6)
- moved M2 84.1 mm to (84.8, 142.0)
- moved M4 79.1 mm to (84.8, 91.2)
- moved J3 54.9 mm to (109.0, 144.3), turned to 180 degrees
- moved M3 52.4 mm to (156.0, 142.0)
- moved J2 49.2 mm to (124.7, 143.5), turned to 180 degrees
- moved SW1 29.9 mm to (118.6, 90.9)
- moved P1 27.4 mm to (101.9, 90.9), turned to 90 degrees
- moved M1 1.09 mm to (156.0, 91.2)
Other:
- board outline added: 80.8 x 60.5 mm

Commit message: Edit PCB
Parts:
- C1, C10, C11, C12, C13, C14, C15, C16, C17, C18, C19, C2, C20, C21, C22, C3, C4, C5, C6, C7, C8, C9, D1, D10, D2, D3, D4, D5, D6, D7, D8, D9, F1, J4, JP1, L1, L2, R1, R10, R11, R12, R13, R14, R15, R16, R17, R18, R19, R2, R20, R21, R24, R25, R26, R3, R4, R5, R6, R7, R8, R9, U1, U2, U3: moved to B.Cu
- moved J1 101.5 mm to (134.0, 142.2), turned to 90 degrees
- moved R15 89.6 mm to (90.0, -3.14)
- moved R5 88.1 mm to (94.4, -2.30)
- moved R4 87.9 mm to (98.8, -2.24)
- moved C4 84.0 mm to (90.0, -0.16)
- moved R3 82.5 mm to (94.4, 0.65)
- moved R13 82.4 mm to (98.8, 0.71)
- moved U2 78.0 mm to (82.2, 3.08), turned to -90 degrees
- moved C5 77.0 mm to (94.2, 3.63)
- moved R1 77.0 mm to (98.6, 3.66)
- moved R9 75.0 mm to (103.0, 4.70)
- moved D2 72.6 mm to (85.1, 114.3), turned to 180 degrees
- moved C1 71.5 mm to (94.2, 6.64)
- moved C3 71.5 mm to (98.6, 6.64)
- moved R11 69.7 mm to (103.0, 7.65)
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Other:
- board size 80.8 x 60.5 mm -> 80.8 x 70.6 mm

Commit message: Edit PCB
Parts:
- R22, R23, X1: moved to B.Cu
- R4: footprint Resistor_SMD:R_0805_2012Metric -> Resistor_SMD:R_0805_2012Metric_Pad1.20x1.40mm_HandSolder; moved to F.Cu
- moved F1 135.4 mm to (103.6, 135.1), turned to -90 degrees
- moved R15 124.6 mm to (89.3, 121.5)
- moved U2 120.4 mm to (66.3, 122.4), turned to 180 degrees
- moved R5 117.0 mm to (115.3, 112.8), turned to 90 degrees
- moved R4 116.7 mm to (125.0, 111.5)
- moved R13 113.2 mm to (89.3, 113.5)
- moved R14 110.5 mm to (89.3, 117.5)
- moved C7 107.5 mm to (64.8, 116.3)
- moved C5 106.8 mm to (120.1, 107.2)
- moved C1 106.6 mm to (119.4, 110.2), turned to -90 degrees
- moved C4 105.4 mm to (105.2, 104.1), turned to 90 degrees
- moved R16 103.0 mm to (89.3, 125.5)
- moved C2 102.2 mm to (112.3, 112.1), turned to 180 degrees
- moved C3 101.7 mm to (105.2, 108.2), turned to 90 degrees
- moved R11 98.8 mm to (89.3, 105.5)
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Connections:
- net Net-(R10-Pad2) renamed /fuel_gauge/B
- net Net-(R11-Pad2) renamed /fuel_gauge/C
- net Net-(R12-Pad2) renamed /fuel_gauge/D
- net Net-(R13-Pad2) renamed /fuel_gauge/E
- net Net-(R14-Pad2) renamed /fuel_gauge/F
- net Net-(R15-Pad2) renamed /fuel_gauge/G
- net Net-(R16-Pad2) renamed /fuel_gauge/H
- net Net-(R9-Pad2) renamed /fuel_gauge/A
Routing:
- net /battery_pack/Battery+: track 0.00 -> 89.6 mm, vias 0 -> 5
- net Net-(C12-Pad1): track 0.00 -> 23.2 mm, vias 0 -> 2
- net /power_input/PV+: track 0.00 -> 17.3 mm
- net Net-(C19-Pad1): track 0.00 -> 9.14 mm
- net Net-(C3-Pad2): track 0.00 -> 8.71 mm
- net Net-(C3-Pad1): track 0.00 -> 8.69 mm
- net Net-(JP1-Pad2): track 0.00 -> 6.49 mm
- net Net-(C18-Pad1): track 0.00 -> 5.65 mm
- net Net-(C9-Pad1): track 0.00 -> 5.48 mm
- net Net-(C10-Pad2): track 0.00 -> 5.45 mm
- net Net-(C10-Pad1): track 0.00 -> 5.45 mm
- net Net-(D9-Pad2): track 0.00 -> 3.86 mm
- net +3V3: track 0.00 -> 3.71 mm
- net GND: track 0.00 -> 3.15 mm
- net /battery_pack/Battery-: track 0.00 -> 3.15 mm
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- added copper zone on B.Cu, net +3V3
- added copper zone on B.Cu, net /battery_pack/Battery+
- added copper zone on B.Cu, net /battery_pack/Battery-
- added copper zone on B.Cu, net /power_input/PV+
- added copper zone on B.Cu, net Net-(C12-Pad1)
- added copper zone on B.Cu, net Net-(D9-Pad2)
- added copper zone on B.Cu, net Net-(L2-Pad1)
- added copper zone on B.Cu, net Net-(L2-Pad2)

Commit message: Edit PCB
Parts:
- J4: moved to F.Cu
- moved J4 60.7 mm to (109.9, 80.6), turned to 90 degrees
- moved SW1 3.03 mm to (101.2, 81.9)
- moved P1 1.78 mm to (119.9, 80.6)
- moved R10 1.27 mm to (88.0, 101.5)
- moved R11 1.27 mm to (88.0, 105.5)
- moved R12 1.27 mm to (88.0, 109.5)
- moved R13 1.27 mm to (88.0, 113.5)
- moved R14 1.27 mm to (88.0, 117.5)
- moved R15 1.27 mm to (88.0, 121.5)
- moved R16 1.27 mm to (88.0, 125.5)
- moved R9 1.27 mm to (88.0, 97.5)
- moved D1 1.27 mm to (83.6, 97.5)
- moved D2 1.27 mm to (83.6, 101.5)
- moved D3 1.27 mm to (83.6, 105.5)
- moved D4 1.27 mm to (83.6, 109.5)
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Connections:
- C2 pad 1: Net-(C2-Pad1) -> /battery_pack/NTC2
- R4 pad 1: Net-(C2-Pad1) -> /battery_pack/NTC2
- R4 pad 2: Net-(R4-Pad2) -> /battery_pack/NTC1
- R5 pad 2: Net-(C2-Pad1) -> /battery_pack/NTC2
- U1 pad 11: Net-(R4-Pad2) -> /battery_pack/NTC1
- U1 pad 7: Net-(C2-Pad1) -> /battery_pack/NTC2

Commit message: Edit PCB
Parts:
- moved C7 43.2 mm to (98.3, 89.2)
- moved U2 43.2 mm to (99.8, 95.2)
- moved R2 16.6 mm to (110.7, 85.6)
- moved R3 2.03 mm to (118.0, 85.1)
- moved R1 1.63 mm to (121.9, 85.1)
- moved J4 0.13 mm to (109.7, 80.6)
Routing:
- net +3V3: track 3.71 -> 152.7 mm, vias 0 -> 3
- net /fuel_gauge/CHARGE_CTRL: track 0.00 -> 86.0 mm, vias 0 -> 5
- net /battery_pack/NTC1: track 0.00 -> 61.4 mm, vias 0 -> 2
- net Net-(R5-Pad1): track 0.00 -> 60.8 mm, vias 0 -> 2
- net /battery_pack/NTC2: track 0.00 -> 49.7 mm, vias 0 -> 1
- net /fuel_gauge/H: track 0.00 -> 39.0 mm, vias 0 -> 2
- net /battery_pack/Battery+: track 89.6 -> 124.1 mm, vias 5 -> 7
- net Net-(SW1-Pad2): track 0.00 -> 34.4 mm, vias 0 -> 2
- net /fuel_gauge/G: track 0.00 -> 34.2 mm, vias 0 -> 2
- net /fuel_gauge/I2C_SCL: track 0.00 -> 31.9 mm
- net /fuel_gauge/I2C_SDA: track 0.00 -> 31.6 mm
- net /fuel_gauge/P1: track 0.00 -> 30.8 mm, vias 0 -> 2
- net /fuel_gauge/F: track 0.00 -> 28.3 mm, vias 0 -> 2
- net /fuel_gauge/D: track 0.00 -> 27.4 mm, vias 0 -> 2
- net /fuel_gauge/C: track 0.00 -> 25.2 mm, vias 0 -> 2
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- added copper zone on B.Cu, net GND
- added copper zone on F.Cu, net GND
Other:
- board text added: "0%"
- board text added: "100%"
- board text added: "3V3"
- board text added: "BATTERY"
- board text added: "Battery Status"
- board text added: "CHARGE EN"
- board text added: "GND"
- board text added: "I2C"
- board text added: "MAX 2,75V!!"
- board text added: "MLAB.CZ 2022"
- board text added: "OUT 3V3"
- board text added: "PV+"
- board text added: "PV-"
- board text added: "SCL"
- board text added: "SDA"
- board text added: "SOLARMINIBAT01A"
- board text added: "Solar Cell In"

Commit message: Edit PCB
Routing:
- net /fuel_gauge/F: track 28.3 -> 27.2 mm
- net /fuel_gauge/G: track 34.2 -> 33.4 mm
- net GND: vias 10 -> 345

Commit message: Edit PCB
Routing:
- net GND: vias 345 -> 350
