File: hw/sch_pcb/battery_pack.kicad_sch (KiCad schematic)
At the start: 0 parts

Commit message: Adding input switching regulator.
Parts:
- added BT? (x4): LTO1865-13, symbol Device:Battery_Cell
Connections:
- new net Battery+: BT?.1 (+), BT?.1 (+), BT?.1 (+), BT?.1 (+)
- new net Battery-: BT?.2 (-), BT?.2 (-), BT?.2 (-), BT?.2 (-)
Other:
- note added: "BATTERY PACK"
Changed lines of the file:
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@@
 (kicad_sch (version 20211123) (generator eeschema)
   (paper "A4")
+  (junction (at 140.335 106.045) (diameter 0) (color 0 0 0 0)
+  )
+  (junction (at 140.335 88.9) (diameter 0) (color 0 0 0 0)
+  )
+  (junction (at 121.285 106.045) (diameter 0) (color 0 0 0 0)
+  )
+  (junction (at 121.285 88.9) (diameter 0) (color 0 0 0 0)
+  )
+  (wire (pts (xy 160.02 88.9) (xy 160.02 93.345))
+    (stroke (width 0) (type default) (color 0 0 0 0))
+  )
+  (wire (pts (xy 121.285 100.965) (xy 121.285 106.045))
+    (stroke (width 0) (type default) (color 0 0 0 0))
+  )
+  (wire (pts (xy 101.6 106.045) (xy 121.285 106.045))
+    (stroke (width 0) (type default) (color 0 0 0 0))
+  )
+  (wire (pts (xy 121.285 88.9) (xy 121.285 93.345))
+    (stroke (width 0) (type default) (color 0 0 0 0))
+  )
+  (wire (pts (xy 140.335 106.045) (xy 160.02 106.045))
+    (stroke (width 0) (type default) (color 0 0 0 0))
+  )
+  (wire (pts (xy 121.285 106.045) (xy 140.335 106.045))
+    (stroke (width 0) (type default) (color 0 0 0 0))
+  )
+  (wire (pts (xy 121.285 79.375) (xy 130.175 79.375))
+    (stroke (width 0) (type default) (color 0 0 0 0))
+  )
+  (wire (pts (xy 121.285 88.9) (xy 121.285 79.375))
+    (stroke (width 0) (type default) (color 0 0 0 0))
+  )
+  (wire (pts (xy 121.285 115.57) (xy 131.445 115.57))
+    (stroke (width 0) (type default) (color 0 0 0 0))
+  )
+  (wire (pts (xy 140.335 88.9) (xy 140.335 93.345))
+    (stroke (width 0) (type default) (color 0 0 0 0))
+  )
+  (wire (pts (xy 101.6 93.345) (xy 101.6 88.9))
+    (stroke (width 0) (type default) (color 0 0 0 0))
+  )
+  (wire (pts (xy 121.285 88.9) (xy 140.335 88.9))
+    (stroke (width 0) (type default) (color 0 0 0 0))
+  )
+  (wire (pts (xy 140.335 100.965) (xy 140.335 106.045))
+    (stroke (width 0) (type default) (color 0 0 0 0))
+  )
+  (wire (pts (xy 121.285 106.045) (xy 121.285 115.57))
+    (stroke (width 0) (type default) (color 0 0 0 0))
+  )
+  (wire (pts (xy 160.02 106.045) (xy 160.02 100.965))
+    (stroke (width 0) (type default) (color 0 0 0 0))
+  )
+  (wire (pts (xy 101.6 100.965) (xy 101.6 106.045))
+    (stroke (width 0) (type default) (color 0 0 0 0))
+  )
+  (wire (pts (xy 140.335 88.9) (xy 160.02 88.9))
+    (stroke (width 0) (type default) (color 0 0 0 0))
+  )
+  (wire (pts (xy 101.6 88.9) (xy 121.285 88.9))
+    (stroke (width 0) (type default) (color 0 0 0 0))
+  )
+  (text "BATTERY PACK" (at 116.205 40.005 0)
+    (effects (font (size 2.9972 2.9972)) (justify left bottom))
+  )
+  (hierarchical_label "Battery+" (shape input) (at 130.175 79.375 0)
+    (effects (font (size 1.524 1.524)) (justify left))
+  )
+  (hierarchical_label "Battery-" (shape input) (at 131.445 115.57 0)
+    (effects (font (size 1.524 1.524)) (justify left))
+  )
+  (symbol (lib_id "Device:Battery_Cell") (at 140.335 98.425 0) (unit 1)
+    (in_bom yes) (on_board yes) (fields_autoplaced)
+    (property "Reference" "BT?" (id 0) (at 143.256 95.5583 0)
+      (effects (font (size 1.27 1.27)) (justify left))
+    )
+    (property "Value" "LTO1865-13" (id 1) (at 143.256 98.0952 0)
+      (effects (font (size 1.27 1.27)) (justify left))
+    )
+    (property "Footprint" "" (id 2) (at 140.335 96.901 90)
+      (effects (font (size 1.27 1.27)) hide)
+    )
+    (property "Datasheet" "https://files.gwl.eu/inc/_doc/attach/StoItem/7015/GWL_LTO1865_Rechargeable.pdf" (id 3) (at 140.335 96.901 90)
+      (effects (font (size 1.27 1.27)) hide)
+    )
+    (pin "1")
+    (pin "2")
+  )
+  (symbol (lib_id "Device:Battery_Cell") (at 121.285 98.425 0) (unit 1)
+    (in_bom yes) (on_board yes) (fields_autoplaced)
+    (property "Reference" "BT?" (id 0) (at 124.206 95.5583 0)
+      (effects (font (size 1.27 1.27)) (justify left))
+    )
+    (property "Value" "LTO1865-13" (id 1) (at 124.206 98.0952 0)
+      (effects (font (size 1.27 1.27)) (justify left))
+    )
+    (property "Footprint" "" (id 2) (at 121.285 96.901 90)
+      (effects (font (size 1.27 1.27)) hide)
+    )
+    (property "Datasheet" "https://files.gwl.eu/inc/_doc/attach/StoItem/7015/GWL_LTO1865_Rechargeable.pdf" (id 3) (at 121.285 96.901 90)
+      (effects (font (size 1.27 1.27)) hide)
+    )
+    (pin "1")
+    (pin "2")
+  )
+  (symbol (lib_id "Device:Battery_Cell") (at 160.02 98.425 0) (unit 1)
+    (in_bom yes) (on_board yes) (fields_autoplaced)
+    (property "Reference" "BT?" (id 0) (at 162.941 95.5583 0)
+      (effects (font (size 1.27 1.27)) (justify left))
+    )
+    (property "Value" "LTO1865-13" (id 1) (at 162.941 98.0952 0)
+      (effects (font (size 1.27 1.27)) (justify left))
+    )
+    (property "Footprint" "" (id 2) (at 160.02 96.901 90)
+      (effects (font (size 1.27 1.27)) hide)
+    )
+    (property "Datasheet" "https://files.gwl.eu/inc/_doc/attach/StoItem/7015/GWL_LTO1865_Rechargeable.pdf" (id 3) (at 160.02 96.901 90)
+      (effects (font (size 1.27 1.27)) hide)
+    )
+    (pin "1")
+    (pin "2")
+  )
+  (symbol (lib_id "Device:Battery_Cell") (at 101.6 98.425 0) (unit 1)
+    (in_bom yes) (on_board yes) (fields_autoplaced)
+    (property "Reference" "BT?" (id 0) (at 104.521 95.5583 0)
+      (effects (font (size 1.27 1.27)) (justify left))
+    )
+    (property "Value" "LTO1865-13" (id 1) (at 104.521 98.0952 0)
+      (effects (font (size 1.27 1.27)) (justify left))
+    )
+    (property "Footprint" "" (id 2) (at 101.6 96.901 90)
+      (effects (font (size 1.27 1.27)) hide)
+    )
+    (property "Datasheet" "https://files.gwl.eu/inc/_doc/attach/StoItem/7015/GWL_LTO1865_Rechargeable.pdf" (id 3) (at 101.6 96.901 90)
+      (effects (font (size 1.27 1.27)) hide)
+    )
+    (pin "1")
+    (pin "2")
+  )
 )

Commit message: Update schematics: Adding datasheet Update title blocks Update pull-up value for CHARGE_CTRL signal.
Other:
- company: (none) -> MLAB.cz
- title: (none) -> SOLARMINIBAT01A
Changed lines of the file:
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@@
   (paper "A4")
   (title_block
+    (title "SOLARMINIBAT01A")
     (date "2022-07-20")
+    (rev "A")
+    (company "MLAB.cz")
     (comment 2 "Solar charged LTO Battery Managment System")
   )

Commit message: Edit schema
Parts:
- added F1: 1,1A, Fuse:Fuse_1812_4532Metric_Pad1.30x3.40mm_HandSolder, symbol Device:Polyfuse
- added J1: HEADER_2x03_PARALLEL, Mlab_Pin_Headers:Straight_2x03, symbol MLAB_HEADER:HEADER_2x03_PARALLEL
- gave numbers to parts that had none: 4
Connections:
- net Battery+: now also F1.1
- new net: F1.2, J1.3, J1.4
- new net GND: J1.1, J1.2, J1.5, J1.6
Changed lines of the file:
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@@
   (junction (at 121.285 88.9) (diameter 0) (color 0 0 0 0)
   )
+  (junction (at 219.075 97.155) (diameter 0) (color 0 0 0 0)
+  )
   (wire (pts (xy 160.02 88.9) (xy 160.02 93.345))
     (stroke (width 0) (type default) (color 0 0 0 0))
   )
+  (wire (pts (xy 219.075 97.155) (xy 222.25 97.155))
+    (stroke (width 0) (type default) (color 0 0 0 0))
+  )
+  (wire (pts (xy 216.535 94.615) (xy 222.25 94.615))
+    (stroke (width 0) (type default) (color 0 0 0 0))
+  )
   (wire (pts (xy 121.285 100.965) (xy 121.285 106.045))
     (stroke (width 0) (type default) (color 0 0 0 0))
@@
     (stroke (width 0) (type default) (color 0 0 0 0))
   )
+  (wire (pts (xy 219.075 97.155) (xy 219.075 99.695))
+    (stroke (width 0) (type default) (color 0 0 0 0))
+  )
+  (wire (pts (xy 207.645 94.615) (xy 208.915 94.615))
+    (stroke (width 0) (type default) (color 0 0 0 0))
+  )
   (wire (pts (xy 121.285 88.9) (xy 121.285 79.375))
     (stroke (width 0) (type default) (color 0 0 0 0))
@@
     (stroke (width 0) (type default) (color 0 0 0 0))
   )
+  (wire (pts (xy 219.075 92.075) (xy 219.075 97.155))
+    (stroke (width 0) (type default) (color 0 0 0 0))
+  )
   (wire (pts (xy 160.02 106.045) (xy 160.02 100.965))
     (stroke (width 0) (type default) (color 0 0 0 0))
@@
   )
   (wire (pts (xy 101.6 88.9) (xy 121.285 88.9))
+    (stroke (width 0) (type default) (color 0 0 0 0))
+  )
+  (wire (pts (xy 222.25 92.075) (xy 219.075 92.075))
     (stroke (width 0) (type default) (color 0 0 0 0))
   )
@@
     (effects (font (size 2.9972 2.9972)) (justify left bottom))
   )
+  (hierarchical_label "Battery+" (shape input) (at 207.645 94.615 180)
+    (effects (font (size 1.524 1.524)) (justify right))
+  )
   (hierarchical_label "Battery+" (shape input) (at 130.175 79.375 0)
     (effects (font (size 1.524 1.524)) (justify left))
@@
   (symbol (lib_id "Device:Battery_Cell") (at 140.335 98.425 0) (unit 1)
     (in_bom yes) (on_board yes) (fields_autoplaced)
-    (property "Reference" "BT?" (id 0) (at 143.256 95.5583 0)
+    (property "Reference" "BT3" (id 0) (at 143.256 95.5583 0)
       (effects (font (size 1.27 1.27)) (justify left))
     )
@@
   (symbol (lib_id "Device:Battery_Cell") (at 121.285 98.425 0) (unit 1)
     (in_bom yes) (on_board yes) (fields_autoplaced)
-    (property "Reference" "BT?" (id 0) (at 124.206 95.5583 0)
+    (property "Reference" "BT2" (id 0) (at 124.206 95.5583 0)
       (effects (font (size 1.27 1.27)) (justify left))
     )
@@
   (symbol (lib_id "Device:Battery_Cell") (at 160.02 98.425 0) (unit 1)
     (in_bom yes) (on_board yes) (fields_autoplaced)
-    (property "Reference" "BT?" (id 0) (at 162.941 95.5583 0)
+    (property "Reference" "BT4" (id 0) (at 162.941 95.5583 0)
       (effects (font (size 1.27 1.27)) (justify left))
     )
@@
     (pin "2")
   )
+  (symbol (lib_id "MLAB_HEADER:HEADER_2x03_PARALLEL") (at 228.6 94.615 0) (unit 1)
+    (in_bom yes) (on_board yes) (fields_autoplaced)
+    (property "Reference" "J1" (id 0) (at 231.775 93.5503 0)
+      (effects (font (size 1.524 1.524)) (justify left))
+    )
+    (property "Value" "HEADER_2x03_PARALLEL" (id 1) (at 231.775 96.8293 0)
+      (effects (font (size 1.524 1.524)) (justify left))
+    )
+    (property "Footprint" "Mlab_Pin_Headers:Straight_2x03" (id 2) (at 228.6 92.075 0)
+      (effects (font (size 1.524 1.524)))
+    )
+    (property "Datasheet" "" (id 3) (at 228.6 92.075 0)
+      (effects (font (size 1.524 1.524)))
+    )
+    (pin "1")
+    (pin "2")
+    (pin "3")
+    (pin "4")
+    (pin "5")
+    (pin "6")
+  )
   (symbol (lib_id "Device:Battery_Cell") (at 101.6 98.425 0) (unit 1)
     (in_bom yes) (on_board yes) (fields_autoplaced)
-    (property "Reference" "BT?" (id 0) (at 104.521 95.5583 0)
+    (property "Reference" "BT1" (id 0) (at 104.521 95.5583 0)
       (effects (font (size 1.27 1.27)) (justify left))
     )
@@
       (effects (font (size 1.27 1.27)) hide)
     )
+    (pin "1")
+    (pin "2")
+  )
+  (symbol (lib_id "power:GND") (at 219.075 99.695 0) (unit 1)
+    (in_bom yes) (on_board yes) (fields_autoplaced)
+    (property "Reference" "#PWR0116" (id 0) (at 219.075 106.045 0)
+      (effects (font (size 1.27 1.27)) hide)
+    )
+    (property "Value" "GND" (id 1) (at 219.075 104.2575 0))
+    (property "Footprint" "" (id 2) (at 219.075 99.695 0)
+      (effects (font (size 1.27 1.27)) hide)
+    )
+    (property "Datasheet" "" (id 3) (at 219.075 99.695 0)
+      (effects (font (size 1.27 1.27)) hide)
+    )
+    (pin "1")
+  )
+  (symbol (lib_id "Device:Polyfuse") (at 212.725 94.615 90) (unit 1)
+    (in_bom yes) (on_board yes) (fields_autoplaced)
+    (property "Reference" "F1" (id 0) (at 212.725 89.2515 90))
+    (property "Value" "1,1A" (id 1) (at 212.725 92.0266 90))
+    (property "Footprint" "Fuse:Fuse_1812_4532Metric_Pad1.30x3.40mm_HandSolder" (id 2) (at 217.805 93.345 0)
+      (effects (font (size 1.27 1.27)) (justify left) hide)
+    )
+    (property "Datasheet" "~" (id 3) (at 212.725 94.615 0)
+      (effects (font (size 1.27 1.27)) hide)
+    )

Commit message: Edit PCB
Parts:
- removed BT1, BT2, BT3, BT4: LTO1865-13, symbol Device:Battery_Cell
- added BT1: 4xLTO18650, Mlab_Batery:4XLTO1865V01A, symbol MLAB_BATERY:4xLTO18650
Connections:
- net Battery+: now also BT1.1 (+)
- net Battery-: now also BT1.2 (-)
- net GND: now also BT1.3 (GND)
Changed lines of the file:
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@@
     (comment 2 "Solar charged LTO Battery Managment System")
   )
-  (junction (at 140.335 106.045) (diameter 0) (color 0 0 0 0)
-  )
-  (junction (at 140.335 88.9) (diameter 0) (color 0 0 0 0)
-  )
-  (junction (at 121.285 106.045) (diameter 0) (color 0 0 0 0)
-  )
-  (junction (at 121.285 88.9) (diameter 0) (color 0 0 0 0)
-  )
   (junction (at 219.075 97.155) (diameter 0) (color 0 0 0 0)
-  )
-  (wire (pts (xy 160.02 88.9) (xy 160.02 93.345))
-    (stroke (width 0) (type default) (color 0 0 0 0))
   )
   (wire (pts (xy 219.075 97.155) (xy 222.25 97.155))
@@
     (stroke (width 0) (type default) (color 0 0 0 0))
   )
-  (wire (pts (xy 121.285 100.965) (xy 121.285 106.045))
-    (stroke (width 0) (type default) (color 0 0 0 0))
-  )
-  (wire (pts (xy 101.6 106.045) (xy 121.285 106.045))
-    (stroke (width 0) (type default) (color 0 0 0 0))
-  )
-  (wire (pts (xy 121.285 88.9) (xy 121.285 93.345))
-    (stroke (width 0) (type default) (color 0 0 0 0))
-  )
-  (wire (pts (xy 140.335 106.045) (xy 160.02 106.045))
-    (stroke (width 0) (type default) (color 0 0 0 0))
-  )
-  (wire (pts (xy 121.285 106.045) (xy 140.335 106.045))
+  (wire (pts (xy 113.665 102.235) (xy 113.665 103.505))
     (stroke (width 0) (type default) (color 0 0 0 0))
   )
@@
     (stroke (width 0) (type default) (color 0 0 0 0))
   )
-  (wire (pts (xy 121.285 88.9) (xy 121.285 79.375))
+  (wire (pts (xy 121.285 79.375) (xy 121.285 92.075))
     (stroke (width 0) (type default) (color 0 0 0 0))
   )
@@
     (stroke (width 0) (type default) (color 0 0 0 0))
   )
-  (wire (pts (xy 140.335 88.9) (xy 140.335 93.345))
-    (stroke (width 0) (type default) (color 0 0 0 0))
-  )
-  (wire (pts (xy 101.6 93.345) (xy 101.6 88.9))
-    (stroke (width 0) (type default) (color 0 0 0 0))
-  )
-  (wire (pts (xy 121.285 88.9) (xy 140.335 88.9))
-    (stroke (width 0) (type default) (color 0 0 0 0))
-  )
-  (wire (pts (xy 140.335 100.965) (xy 140.335 106.045))
-    (stroke (width 0) (type default) (color 0 0 0 0))
-  )
-  (wire (pts (xy 121.285 106.045) (xy 121.285 115.57))
+  (wire (pts (xy 121.285 102.235) (xy 121.285 115.57))
     (stroke (width 0) (type default) (color 0 0 0 0))
   )
   (wire (pts (xy 219.075 92.075) (xy 219.075 97.155))
-    (stroke (width 0) (type default) (color 0 0 0 0))
-  )
-  (wire (pts (xy 160.02 106.045) (xy 160.02 100.965))
-    (stroke (width 0) (type default) (color 0 0 0 0))
-  )
-  (wire (pts (xy 101.6 100.965) (xy 101.6 106.045))
-    (stroke (width 0) (type default) (color 0 0 0 0))
-  )
-  (wire (pts (xy 140.335 88.9) (xy 160.02 88.9))
-    (stroke (width 0) (type default) (color 0 0 0 0))
-  )
-  (wire (pts (xy 101.6 88.9) (xy 121.285 88.9))
     (stroke (width 0) (type default) (color 0 0 0 0))
   )
@@
     (effects (font (size 1.524 1.524)) (justify left))
   )
-  (symbol (lib_id "Device:Battery_Cell") (at 140.335 98.425 0) (unit 1)
+  (symbol (lib_id "MLAB_BATERY:4xLTO18650") (at 121.285 98.425 0) (unit 1)
     (in_bom yes) (on_board yes) (fields_autoplaced)
-    (property "Reference" "BT3" (id 0) (at 143.256 95.5583 0)
+    (property "Reference" "BT1" (id 0) (at 133.985 96.1195 0)
       (effects (font (size 1.27 1.27)) (justify left))
     )
-    (property "Value" "LTO1865-13" (id 1) (at 143.256 98.0952 0)
+    (property "Value" "4xLTO18650" (id 1) (at 133.985 98.8946 0)
       (effects (font (size 1.27 1.27)) (justify left))
     )
-    (property "Footprint" "" (id 2) (at 140.335 96.901 90)
+    (property "Footprint" "Mlab_Batery:4XLTO1865V01A" (id 2) (at 121.285 96.901 90)
       (effects (font (size 1.27 1.27)) hide)
     )
-    (property "Datasheet" "https://files.gwl.eu/inc/_doc/attach/StoItem/7015/GWL_LTO1865_Rechargeable.pdf" (id 3) (at 140.335 96.901 90)
+    (property "Datasheet" "~" (id 3) (at 121.285 96.901 90)
       (effects (font (size 1.27 1.27)) hide)
     )
     (pin "1")
     (pin "2")
-  )
-  (symbol (lib_id "Device:Battery_Cell") (at 121.285 98.425 0) (unit 1)
-    (in_bom yes) (on_board yes) (fields_autoplaced)
-    (property "Reference" "BT2" (id 0) (at 124.206 95.5583 0)
-      (effects (font (size 1.27 1.27)) (justify left))
-    )
-    (property "Value" "LTO1865-13" (id 1) (at 124.206 98.0952 0)
-      (effects (font (size 1.27 1.27)) (justify left))
-    )
-    (property "Footprint" "" (id 2) (at 121.285 96.901 90)
-      (effects (font (size 1.27 1.27)) hide)
-    )
-    (property "Datasheet" "https://files.gwl.eu/inc/_doc/attach/StoItem/7015/GWL_LTO1865_Rechargeable.pdf" (id 3) (at 121.285 96.901 90)
-      (effects (font (size 1.27 1.27)) hide)
-    )
-    (pin "1")
-    (pin "2")
-  )
-  (symbol (lib_id "Device:Battery_Cell") (at 160.02 98.425 0) (unit 1)
-    (in_bom yes) (on_board yes) (fields_autoplaced)
-    (property "Reference" "BT4" (id 0) (at 162.941 95.5583 0)
-      (effects (font (size 1.27 1.27)) (justify left))
-    )
-    (property "Value" "LTO1865-13" (id 1) (at 162.941 98.0952 0)
-      (effects (font (size 1.27 1.27)) (justify left))
-    )
-    (property "Footprint" "" (id 2) (at 160.02 96.901 90)
-      (effects (font (size 1.27 1.27)) hide)
-    )
-    (property "Datasheet" "https://files.gwl.eu/inc/_doc/attach/StoItem/7015/GWL_LTO1865_Rechargeable.pdf" (id 3) (at 160.02 96.901 90)
-      (effects (font (size 1.27 1.27)) hide)
-    )
-    (pin "1")
-    (pin "2")
+    (pin "3")
   )
   (symbol (lib_id "MLAB_HEADER:HEADER_2x03_PARALLEL") (at 228.6 94.615 0) (unit 1)
@@
     )
     (property "Footprint" "Mlab_Pin_Headers:Straight_2x03" (id 2) (at 228.6 92.075 0)
-      (effects (font (size 1.524 1.524)))
+      (effects (font (size 1.524 1.524)) hide)
     )
     (property "Datasheet" "" (id 3) (at 228.6 92.075 0)
@@
     (pin "5")
     (pin "6")
-  )
-  (symbol (lib_id "Device:Battery_Cell") (at 101.6 98.425 0) (unit 1)
-    (in_bom yes) (on_board yes) (fields_autoplaced)
-    (property "Reference" "BT1" (id 0) (at 104.521 95.5583 0)
-      (effects (font (size 1.27 1.27)) (justify left))
-    )
-    (property "Value" "LTO1865-13" (id 1) (at 104.521 98.0952 0)
-      (effects (font (size 1.27 1.27)) (justify left))
-    )
-    (property "Footprint" "" (id 2) (at 101.6 96.901 90)
-      (effects (font (size 1.27 1.27)) hide)
-    )
-    (property "Datasheet" "https://files.gwl.eu/inc/_doc/attach/StoItem/7015/GWL_LTO1865_Rechargeable.pdf" (id 3) (at 101.6 96.901 90)
-      (effects (font (size 1.27 1.27)) hide)
-    )
-    (pin "1")
-    (pin "2")
   )
   (symbol (lib_id "power:GND") (at 219.075 99.695 0) (unit 1)
@@
       (effects (font (size 1.27 1.27)) hide)
     )
+    (pin "1")
+  )
+  (symbol (lib_id "power:GND") (at 113.665 103.505 0) (unit 1)
+    (in_bom yes) (on_board yes) (fields_autoplaced)
+    (property "Reference" "#PWR0141" (id 0) (at 113.665 109.855 0)
+      (effects (font (size 1.27 1.27)) hide)
+    )
+    (property "Value" "GND" (id 1) (at 113.665 108.0675 0))
+    (property "Footprint" "" (id 2) (at 113.665 103.505 0)
+      (effects (font (size 1.27 1.27)) hide)
+    )
+    (property "Datasheet" "" (id 3) (at 113.665 103.505 0)
+      (effects (font (size 1.27 1.27)) hide)
+    )

Commit message: Edit PCB
Connections:
- new net NTC1: BT1.5
- new net NTC2: BT1.6
Changed lines of the file:
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@@
     (effects (font (size 1.524 1.524)) (justify left))
+  )
+  (hierarchical_label "NTC1" (shape input) (at 101.6 100.965 270)
+    (effects (font (size 1.524 1.524)) (justify right))
+  )
+  (hierarchical_label "NTC2" (shape input) (at 105.41 100.965 270)
+    (effects (font (size 1.524 1.524)) (justify right))
   )
   (hierarchical_label "Battery-" (shape input) (at 131.445 115.57 0)
@@
     (pin "2")
     (pin "3")
+    (pin "5")
+    (pin "6")
   )
   (symbol (lib_id "MLAB_HEADER:HEADER_2x03_PARALLEL") (at 228.6 94.615 0) (unit 1)

Commit message: Edit UST ID
Parts:
- F1: UST_ID (none) -> 5c70984512875079b91f88d3
Changed lines of the file:
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@@
+      (effects (font (size 1.27 1.27)) hide)
+    )
+    (property "UST_ID" "5c70984512875079b91f88d3" (id 4) (at 212.725 94.615 0)
       (effects (font (size 1.27 1.27)) hide)
     )
